File: ThumbsUp.kicad_pcb (KiCad board)
At the start: 2 copper layers, 250.8 x 280.8 mm, 169 parts, among them IC1 RP2040, IC2 W25Q128JVSIM, IC3 RP2040, IC4 W25Q128JVSIM, J1 Conn_01x04_Male, J10 Raiser_Male, J11 Raiser_Female, J12 Raiser_Male, J13 Raiser_Female, J14 Raiser_Male, J15 Raiser_Female, J16 Raiser_Male, J17 Raiser_Female, J18 Raiser_Male, J19 Raiser_Female, J2 Conn_01x04_Male, J20 Conn_01x04_Female, J21 Conn_01x04_Female, J22 Conn_01x04_Female, J23 Conn_01x04_Female, J24 Conn_01x04_Male, J25 Conn_01x04_Male, J26 Conn_01x04_Male, J27 Conn_01x04_Male, J28 Conn_01x04_Female, J29 Conn_01x04_Female, J3 Conn_01x04_Female, J30 Conn_01x04_Female, J31 Conn_01x04_Female, J32 USB_C_Receptacle_USB2.0, J33 Raiser_Male, J34 Raiser_Female, J35 Raiser_Male, J36 STX-3501-3N, J37 USB_C_Receptacle_USB2.0, J38 Raiser_Female, J39 Raiser_Male, J4 Conn_01x04_Male, J40 Raiser_Female, J41 Raiser_Male, J42 Raiser_Female, J43 Raiser_Male, J44 Raiser_Female, J45 Raiser_Male, J46 STX-3501-3N, J47 Raiser_Female, J48 Raiser_Male, J49 Raiser_Female, J5 Conn_01x04_Female, J50 Raiser_Male, J51 Raiser_Female, J52 Raiser_Male, J6 Conn_01x04_Male, J7 Conn_01x04_Male, J8 Conn_01x04_Male, J9 Raiser_Female, U1 NCP1117-3.3_SOT223, U2 NCP1117-3.3_SOT223, Y1 ABLS-12.000MHZ-B4-T, Y2 ABLS-12.000MHZ-B4-T

Commit message: Populated DNF resistors with 10K.
Parts:
- R13, R7: value DNF -> 10K
Changed lines of the file:
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@@
       (effects (font (size 1 1) (thickness 0.15)) (justify mirror))
     )
-    (fp_text value DNF (at 0 -1.17) (layer B.Fab)
+    (fp_text value 10K (at 0 -1.17) (layer B.Fab)
       (effects (font (size 1 1) (thickness 0.15)) (justify mirror))
     )
@@
       (effects (font (size 1 1) (thickness 0.15)) (justify mirror))
     )
-    (fp_text value DNF (at 0 -1.17) (layer B.Fab)
+    (fp_text value 10K (at 0 -1.17) (layer B.Fab)
       (effects (font (size 1 1) (thickness 0.15)) (justify mirror))
     )
@@
   (segment (start 182.749038 462.852002) (end 182.722036 462.825) (width 0.2) (layer F.Cu) (net 49))
   (segment (start 182.722036 462.825) (end 174.575 462.825) (width 0.2) (layer F.Cu) (net 49))
-  (segment (start 168.05 466.35) (end 174.82901 466.35) (width 0.2) (layer F.Cu) (net 231))
-  (via (at 174.82901 466.35) (size 0.8) (drill 0.4) (layers F.Cu B.Cu) (net 231))
-  (segment (start 168.05 466.35) (end 168.05 463.98) (width 0.2) (layer B.Cu) (net 231) (status 20))
-  (segment (start 168.05 463.98) (end 168.02 463.95) (width 0.2) (layer B.Cu) (net 231) (status 30))
-  (segment (start 168.07 466.33) (end 168.05 466.35) (width 0.2) (layer B.Cu) (net 231))
-  (via (at 168.05 466.35) (size 0.8) (drill 0.4) (layers F.Cu B.Cu) (net 231))
   (segment (start 180.084574 455.15) (end 178.838587 456.395987) (width 0.2) (layer B.Cu) (net 63))
   (segment (start 178.475 456.4) (end 177.85 456.4) (width 0.2) (layer B.Cu) (net 63) (status 20))
@@
   (segment (start 77.048913 461.418953) (end 75.255634 459.625674) (width 0.2) (layer B.Cu) (net 230))
   (segment (start 75.255634 459.625674) (end 70.873341 459.625674) (width 0.2) (layer B.Cu) (net 230))
+  (segment (start 168.05 466.35) (end 174.82901 466.35) (width 0.2) (layer F.Cu) (net 231))
+  (via (at 174.82901 466.35) (size 0.8) (drill 0.4) (layers F.Cu B.Cu) (net 231))
+  (segment (start 168.05 466.35) (end 168.05 463.98) (width 0.2) (layer B.Cu) (net 231) (status 20))
+  (segment (start 168.05 463.98) (end 168.02 463.95) (width 0.2) (layer B.Cu) (net 231) (status 30))
+  (segment (start 168.07 466.33) (end 168.05 466.35) (width 0.2) (layer B.Cu) (net 231))
+  (via (at 168.05 466.35) (size 0.8) (drill 0.4) (layers F.Cu B.Cu) (net 231))
   (segment (start 214.123921 459.625674) (end 214.098247 459.6) (width 0.2) (layer B.Cu) (net 231))
   (segment (start 181.012537 466.35) (end 174.82901 466.35) (width 0.2) (layer B.Cu) (net 231))
